File: SailbotBMS.sch (KiCad schematic (older format))
At the start: 0 parts

Commit message: renaming and project organization
Parts:
- added BT? (x4): Battery_Cell, symbol Device:Battery_Cell
- added U?: BQ77915, symbol BQ77915:BQ77915
Connections:
- net labels added: VDD, VSS
- wire segments 0 -> 17
Changed lines of the file:
@@
 EESchema Schematic File Version 4
+LIBS:SailbotBMS-cache
 EELAYER 26 0
 EELAYER END
@@
 $EndDescr
 $Comp
-L power:+BATT #PWR?
-U 1 1 5CED8E1B
-P 6500 3000
-F 0 "#PWR?" H 6500 2850 50  0001 C CNN
-F 1 "+BATT" V 6515 3127 50  0000 L CNN
-F 2 "" H 6500 3000 50  0001 C CNN
-F 3 "" H 6500 3000 50  0001 C CNN
-	1    6500 3000
-	0    -1   -1   0
+L BQ77915:BQ77915 U?
+U 1 1 5D24103E
+P 4900 2650
+F 0 "U?" H 4875 3375 50  0000 C CNN
+F 1 "BQ77915" H 4875 3284 50  0000 C CNN
+F 2 "" H 5250 2400 50  0001 C CNN
+F 3 "" H 5250 2400 50  0001 C CNN
+	1    4900 2650
+	1    0    0    -1
 $EndComp
 $Comp
+L Device:Battery_Cell BT?
+U 1 1 5D2410CF
+P 3200 3550
+F 0 "BT?" H 3318 3646 50  0000 L CNN
+F 1 "Battery_Cell" H 3318 3555 50  0000 L CNN
+F 2 "" V 3200 3610 50  0001 C CNN
+F 3 "~" V 3200 3610 50  0001 C CNN
+	1    3200 3550
+	1    0    0    -1
+$EndComp
+$Comp
+L Device:Battery_Cell BT?
+U 1 1 5D241151
+P 3200 3250
+F 0 "BT?" H 3318 3346 50  0000 L CNN
+F 1 "Battery_Cell" H 3318 3255 50  0000 L CNN
+F 2 "" V 3200 3310 50  0001 C CNN
+F 3 "~" V 3200 3310 50  0001 C CNN
+	1    3200 3250
+	1    0    0    -1
+$EndComp
+$Comp
+L Device:Battery_Cell BT?
+U 1 1 5D24116F
+P 3200 2950
+F 0 "BT?" H 3318 3046 50  0000 L CNN
+F 1 "Battery_Cell" H 3318 2955 50  0000 L CNN
+F 2 "" V 3200 3010 50  0001 C CNN
+F 3 "~" V 3200 3010 50  0001 C CNN
+	1    3200 2950
+	1    0    0    -1
+$EndComp
+$Comp
+L Device:Battery_Cell BT?
+U 1 1 5D2411AB
+P 3200 2650
+F 0 "BT?" H 3318 2746 50  0000 L CNN
+F 1 "Battery_Cell" H 3318 2655 50  0000 L CNN
+F 2 "" V 3200 2710 50  0001 C CNN
+F 3 "~" V 3200 2710 50  0001 C CNN
+	1    3200 2650
+	1    0    0    -1
+$EndComp
+Wire Wire Line
+	3200 2450 4450 2450
+Wire Wire Line
+	4450 2550 3850 2550
+Wire Wire Line
+	3850 2550 3850 2750
+Wire Wire Line
+	3850 2750 3200 2750
+Connection ~ 3200 2750
+Wire Wire Line
+	4450 2650 4000 2650
+Wire Wire Line
+	4000 2650 4000 3050
+Wire Wire Line
+	4000 3050 3200 3050
+Connection ~ 3200 3050
+Wire Wire Line
+	4450 2750 4150 2750
+Wire Wire Line
+	4150 2750 4150 3350
+Wire Wire Line
+	4150 3350 3200 3350
+Connection ~ 3200 3350
+Wire Wire Line
+	3200 3650 4300 3650
+Wire Wire Line
+	4300 3650 4300 2850
+Wire Wire Line
+	4300 2850 4450 2850
+$Comp
+L power:+BATT #PWR?
+U 1 1 5D2416AB
+P 3200 2450
+F 0 "#PWR?" H 3200 2300 50  0001 C CNN
+F 1 "+BATT" H 3215 2623 50  0000 C CNN
+F 2 "" H 3200 2450 50  0001 C CNN
+F 3 "" H 3200 2450 50  0001 C CNN
+	1    3200 2450
+	1    0    0    -1
+$EndComp
+Connection ~ 3200 2450
+$Comp
 L power:-BATT #PWR?
-U 1 1 5CED8E89
-P 5150 3000
-F 0 "#PWR?" H 5150 2850 50  0001 C CNN
-F 1 "-BATT" V 5165 3127 50  0000 L CNN
-F 2 "" H 5150 3000 50  0001 C CNN
-F 3 "" H 5150 3000 50  0001 C CNN
-	1    5150 3000
-	0    -1   -1   0
+U 1 1 5D24173B
+P 3200 3650
+F 0 "#PWR?" H 3200 3500 50  0001 C CNN
+F 1 "-BATT" H 3215 3823 50  0000 C CNN
+F 2 "" H 3200 3650 50  0001 C CNN
+F 3 "" H 3200 3650 50  0001 C CNN
+	1    3200 3650
+	-1   0    0    1
 $EndComp
+Connection ~ 3200 3650
+$Comp
+L power:VDD #PWR?
+U 1 1 5D2418CC
+P 4200 2050
+F 0 "#PWR?" H 4200 1900 50  0001 C CNN
+F 1 "VDD" H 4217 2223 50  0000 C CNN
+F 2 "" H 4200 2050 50  0001 C CNN
+F 3 "" H 4200 2050 50  0001 C CNN
+	1    4200 2050
+	1    0    0    -1
+$EndComp
+$Comp
+L power:VSS #PWR?
+U 1 1 5D2419E9
+P 4050 2050
+F 0 "#PWR?" H 4050 1900 50  0001 C CNN
+F 1 "VSS" H 4067 2223 50  0000 C CNN
+F 2 "" H 4050 2050 50  0001 C CNN
+F 3 "" H 4050 2050 50  0001 C CNN
+	1    4050 2050
+	1    0    0    -1
+$EndComp
+Wire Wire Line
+	4200 2050 4200 2150
+Wire Wire Line
+	4450 2150 4200 2150
+Wire Wire Line
+	4050 2050 4050 2950
+Wire Wire Line
+	4050 2950 4450 2950
 $EndSCHEMATC

Commit message: good morning fixes
Parts:
- added C?: C, symbol Device:C
- added Q?: Q_NMOS_DGS, symbol Device:Q_NMOS_DGS
- added Q?: Q_PMOS_DGS, symbol Device:Q_PMOS_DGS
Connections:
- net labels added: 0, GND, GNDPWR, VDDA
- net labels removed: VSS
- wire segments 17 -> 35
Changed lines of the file:
@@
 L Device:Battery_Cell BT?
 U 1 1 5D2410CF
-P 3200 3550
-F 0 "BT?" H 3318 3646 50  0000 L CNN
-F 1 "Battery_Cell" H 3318 3555 50  0000 L CNN
-F 2 "" V 3200 3610 50  0001 C CNN
-F 3 "~" V 3200 3610 50  0001 C CNN
-	1    3200 3550
+P 1900 3550
+F 0 "BT?" H 2018 3646 50  0000 L CNN
+F 1 "Battery_Cell" H 2018 3555 50  0000 L CNN
+F 2 "" V 1900 3610 50  0001 C CNN
+F 3 "~" V 1900 3610 50  0001 C CNN
+	1    1900 3550
 	1    0    0    -1
 $EndComp
@@
 L Device:Battery_Cell BT?
 U 1 1 5D241151
-P 3200 3250
-F 0 "BT?" H 3318 3346 50  0000 L CNN
-F 1 "Battery_Cell" H 3318 3255 50  0000 L CNN
-F 2 "" V 3200 3310 50  0001 C CNN
-F 3 "~" V 3200 3310 50  0001 C CNN
-	1    3200 3250
+P 1900 3250
+F 0 "BT?" H 2018 3346 50  0000 L CNN
+F 1 "Battery_Cell" H 2018 3255 50  0000 L CNN
+F 2 "" V 1900 3310 50  0001 C CNN
+F 3 "~" V 1900 3310 50  0001 C CNN
+	1    1900 3250
 	1    0    0    -1
 $EndComp
@@
 L Device:Battery_Cell BT?
 U 1 1 5D24116F
-P 3200 2950
-F 0 "BT?" H 3318 3046 50  0000 L CNN
-F 1 "Battery_Cell" H 3318 2955 50  0000 L CNN
-F 2 "" V 3200 3010 50  0001 C CNN
-F 3 "~" V 3200 3010 50  0001 C CNN
-	1    3200 2950
+P 1900 2950
+F 0 "BT?" H 2018 3046 50  0000 L CNN
+F 1 "Battery_Cell" H 2018 2955 50  0000 L CNN
+F 2 "" V 1900 3010 50  0001 C CNN
+F 3 "~" V 1900 3010 50  0001 C CNN
+	1    1900 2950
 	1    0    0    -1
 $EndComp
@@
 L Device:Battery_Cell BT?
 U 1 1 5D2411AB
-P 3200 2650
-F 0 "BT?" H 3318 2746 50  0000 L CNN
-F 1 "Battery_Cell" H 3318 2655 50  0000 L CNN
-F 2 "" V 3200 2710 50  0001 C CNN
-F 3 "~" V 3200 2710 50  0001 C CNN
-	1    3200 2650
-	1    0    0    -1
-$EndComp
-Wire Wire Line
-	3200 2450 4450 2450
-Wire Wire Line
-	4450 2550 3850 2550
-Wire Wire Line
-	3850 2550 3850 2750
-Wire Wire Line
-	3850 2750 3200 2750
-Connection ~ 3200 2750
-Wire Wire Line
-	4450 2650 4000 2650
-Wire Wire Line
-	4000 2650 4000 3050
-Wire Wire Line
-	4000 3050 3200 3050
-Connection ~ 3200 3050
-Wire Wire Line
-	4450 2750 4150 2750
-Wire Wire Line
-	4150 2750 4150 3350
-Wire Wire Line
-	4150 3350 3200 3350
-Connection ~ 3200 3350
-Wire Wire Line
-	3200 3650 4300 3650
-Wire Wire Line
-	4300 3650 4300 2850
-Wire Wire Line
-	4300 2850 4450 2850
+P 1900 2650
+F 0 "BT?" H 2018 2746 50  0000 L CNN
+F 1 "Battery_Cell" H 2018 2655 50  0000 L CNN
+F 2 "" V 1900 2710 50  0001 C CNN
+F 3 "~" V 1900 2710 50  0001 C CNN
+	1    1900 2650
+	1    0    0    -1
+$EndComp
 $Comp
 L power:+BATT #PWR?
 U 1 1 5D2416AB
-P 3200 2450
-F 0 "#PWR?" H 3200 2300 50  0001 C CNN
-F 1 "+BATT" H 3215 2623 50  0000 C CNN
-F 2 "" H 3200 2450 50  0001 C CNN
-F 3 "" H 3200 2450 50  0001 C CNN
-	1    3200 2450
-	1    0    0    -1
-$EndComp
-Connection ~ 3200 2450
+P 1900 2450
+F 0 "#PWR?" H 1900 2300 50  0001 C CNN
+F 1 "+BATT" H 1915 2623 50  0000 C CNN
+F 2 "" H 1900 2450 50  0001 C CNN
+F 3 "" H 1900 2450 50  0001 C CNN
+	1    1900 2450
+	1    0    0    -1
+$EndComp
+Connection ~ 1900 2450
 $Comp
 L power:-BATT #PWR?
 U 1 1 5D24173B
-P 3200 3650
-F 0 "#PWR?" H 3200 3500 50  0001 C CNN
-F 1 "-BATT" H 3215 3823 50  0000 C CNN
-F 2 "" H 3200 3650 50  0001 C CNN
-F 3 "" H 3200 3650 50  0001 C CNN
-	1    3200 3650
+P 2100 3650
+F 0 "#PWR?" H 2100 3500 50  0001 C CNN
+F 1 "-BATT" H 2115 3823 50  0000 C CNN
+F 2 "" H 2100 3650 50  0001 C CNN
+F 3 "" H 2100 3650 50  0001 C CNN
+	1    2100 3650
 	-1   0    0    1
 $EndComp
-Connection ~ 3200 3650
 $Comp
 L power:VDD #PWR?
@@
 	1    0    0    -1
 $EndComp
-$Comp
-L power:VSS #PWR?
-U 1 1 5D2419E9
-P 4050 2050
-F 0 "#PWR?" H 4050 1900 50  0001 C CNN
-F 1 "VSS" H 4067 2223 50  0000 C CNN
-F 2 "" H 4050 2050 50  0001 C CNN
-F 3 "" H 4050 2050 50  0001 C CNN
-	1    4050 2050
-	1    0    0    -1
-$EndComp
 Wire Wire Line
 	4200 2050 4200 2150
 Wire Wire Line
 	4450 2150 4200 2150
-Wire Wire Line
-	4050 2050 4050 2950
-Wire Wire Line
-	4050 2950 4450 2950
+$Comp
+L pspice:0 #GND?
+U 1 1 5D242274
+P 5850 2950
+F 0 "#GND?" H 5850 2850 50  0001 C CNN
+F 1 "0" H 5850 3037 50  0000 C CNN
+F 2 "" H 5850 2950 50  0001 C CNN
+F 3 "" H 5850 2950 50  0001 C CNN
+	1    5850 2950
+	1    0    0    -1
+$EndComp
+Wire Wire Line
+	5850 2950 5300 2950
+$Comp
+L power:GNDPWR #PWR?
+U 1 1 5D248051
+P 4250 2950
+F 0 "#PWR?" H 4250 2750 50  0001 C CNN
+F 1 "GNDPWR" H 4254 2796 50  0000 C CNN
+F 2 "" H 4250 2900 50  0001 C CNN
+F 3 "" H 4250 2900 50  0001 C CNN
+	1    4250 2950
+	1    0    0    -1
+$EndComp
+$Comp
+L Device:C C?
+U 1 1 5D248E8E
+P 3600 2100
+F 0 "C?" H 3715 2146 50  0000 L CNN
+F 1 "C" H 3715 2055 50  0000 L CNN
+F 2 "" H 3638 1950 50  0001 C CNN
+F 3 "~" H 3600 2100 50  0001 C CNN
+	1    3600 2100
+	1    0    0    -1
+$EndComp
+Wire Wire Line
+	1900 2450 4450 2450
+Wire Wire Line
+	4250 2950 4450 2950
+Wire Wire Line
+	1900 2750 2500 2750
+Wire Wire Line
+	2500 2750 2500 2550
+Wire Wire Line
+	2500 2550 4450 2550
+Connection ~ 1900 2750
+Wire Wire Line
+	1900 3050 2550 3050
+Wire Wire Line
+	2550 3050 2550 2650
+Wire Wire Line
+	2550 2650 4450 2650
+Connection ~ 1900 3050
+Wire Wire Line
+	1900 3350 2600 3350
+Wire Wire Line
+	2600 3350 2600 2750
+Wire Wire Line
+	2600 2750 4450 2750
+Connection ~ 1900 3350
+Wire Wire Line
+	2650 2850 4450 2850
+$Comp
+L power:VDDA #PWR?
+U 1 1 5D24A158
+P 2950 2250
+F 0 "#PWR?" H 2950 2100 50  0001 C CNN
+F 1 "VDDA" V 2968 2378 50  0000 L CNN
+F 2 "" H 2950 2250 50  0001 C CNN
+F 3 "" H 2950 2250 50  0001 C CNN
+	1    2950 2250
+	0    -1   -1   0
+$EndComp
+Wire Wire Line
+	4450 2250 3600 2250
+Connection ~ 3600 2250
+Wire Wire Line
+	3600 2250 3150 2250
+$Comp
+L power:GND #PWR?
+U 1 1 5D24A43F
+P 3350 2050
+F 0 "#PWR?" H 3350 1800 50  0001 C CNN
+F 1 "GND" H 3355 1877 50  0000 C CNN
+F 2 "" H 3350 2050 50  0001 C CNN
+F 3 "" H 3350 2050 50  0001 C CNN
+	1    3350 2050
+	1    0    0    -1
+$EndComp
+Wire Wire Line
+	3350 2050 3350 1950
+Wire Wire Line
+	3350 1950 3600 1950
+Wire Wire Line
+	3150 2250 3150 1750
+Wire Wire Line
+	3150 1750 5550 1750
+Wire Wire Line
+	5550 1750 5550 2550
+Wire Wire Line
+	5550 2550 5300 2550
+Connection ~ 3150 2250
+Wire Wire Line
+	3150 2250 2950 2250
+$Comp
+L Device:Q_NMOS_DGS Q?
+U 1 1 5D24BC09
+P 4350 4400
+F 0 "Q?" V 4600 4400 50  0000 C CNN
+F 1 "Q_NMOS_DGS" V 4691 4400 50  0000 C CNN
+F 2 "" H 4550 4500 50  0001 C CNN
+F 3 "~" H 4350 4400 50  0001 C CNN
+	1    4350 4400
+	0    1    1    0
+$EndComp
+$Comp
+L Device:Q_PMOS_DGS Q?
+U 1 1 5D24BCAC
+P 5350 4400
+F 0 "Q?" V 5600 4400 50  0000 C CNN
+F 1 "Q_PMOS_DGS" V 5691 4400 50  0000 C CNN
+F 2 "" H 5550 4500 50  0001 C CNN
+F 3 "~" H 5350 4400 50  0001 C CNN
+	1    5350 4400
+	0    1    1    0
+$EndComp
+Wire Wire Line
+	5300 3250 5350 3250
+Wire Wire Line
+	5350 3250 5350 4200
+Wire Wire Line
+	4450 3250 4350 3250
+Wire Wire Line
+	4350 3250 4350 4200
+Wire Wire Line
+	5150 4500 4550 4500
+Wire Wire Line
+	1900 4500 4150 4500
+Wire Wire Line
+	1900 3650 2100 3650
+Wire Wire Line
+	2650 2850 2650 3650
+Wire Wire Line
+	1900 3650 1900 4500
+Connection ~ 1900 3650
+Connection ~ 2100 3650
+Wire Wire Line
+	2100 3650 2650 3650
+Wire Wire Line
+	4450 2350 4450 2450
+Connection ~ 4450 2450
 $EndSCHEMATC

Commit message: initial inplementation functionality
Parts:
- removed BT? (x4): Battery_Cell, symbol Device:Battery_Cell
- removed C?: C, symbol Device:C
- removed Q?: Q_PMOS_DGS, symbol Device:Q_PMOS_DGS
- added C? (x6), C_VDO: C, symbol Device:C
- added J?: Conn_01x05_Female, symbol Connector:Conn_01x05_Female
- added Q?: Q_NMOS_DGS, symbol Device:Q_NMOS_DGS
- added RN?: R_Pack05, symbol Device:R_Pack05
- added R_CB, R_CHG, R_DSG, R_GS (x2), R_LD, R_OCD, R_SNS, R_TS_PU, R_VDD: R, symbol Device:R
- added TH?: Thermistor, symbol Device:Thermistor
Connections:
- net labels added: GNDREF, PACK+, PACK-, PRES
- net labels removed: +BATT, -BATT, 0, GND, GNDPWR, VDD, VDDA
- wire segments 35 -> 100

Commit message: end of day commit
Parts:
- removed RN?: R_Pack05, symbol Device:R_Pack05
- added J2: Conn_01x02, TerminalBlock_Phoenix:TerminalBlock_Phoenix_MKDS-1,5-2-5.08_1x02_P5.08mm_Horizontal, symbol Connector_Generic:Conn_01x02
- added J3: Conn_01x02, Connector_PinHeader_2.54mm:PinHeader_1x02_P2.54mm_Vertical, symbol Connector_Generic:Conn_01x02
- added R1, R2, R3, R4, R5: 33, Resistor_SMD:R_0603_1608Metric, symbol Device:R
- C1, C2, C3, C4, C5, C_VDD1: renamed from C?; value C -> 1uF; footprint (none) -> Capacitor_SMD:C_0603_1608Metric
- C_VDO1: renamed from C_VDO; value C -> 1uF; footprint (none) -> Capacitor_SMD:C_0603_1608Metric
- J1: renamed from J?; footprint (none) -> Connector_JST:JST_XH_B05B-XH-AM_1x05_P2.50mm_Vertical
- Q_NMOS_CHG1: renamed from Q?; value Q_NMOS_DGS -> Q2
- Q_NMOS_DGS1: renamed from Q?; value Q_NMOS_DGS -> Q
- R_CB1: renamed from R_CB; value R -> 10k; footprint (none) -> Resistor_SMD:R_0603_1608Metric
- R_CHG1: renamed from R_CHG; footprint (none) -> Resistor_SMD:R_0603_1608Metric
- R_DSG1: renamed from R_DSG; footprint (none) -> Resistor_SMD:R_0603_1608Metric
- R_GS1, R_GS2: renamed from R_GS; value R -> 1M; footprint (none) -> Resistor_SMD:R_0603_1608Metric
- R_LD1: renamed from R_LD; value R -> 470k; footprint (none) -> Resistor_SMD:R_0603_1608Metric
- R_OCD1: renamed from R_OCD; footprint (none) -> Resistor_SMD:R_0603_1608Metric
- R_SNS1: renamed from R_SNS; value R -> 100m; footprint (none) -> Resistor_SMD:R_0603_1608Metric
- R_TS_PU1: renamed from R_TS_PU; value R -> 10k; footprint (none) -> Resistor_SMD:R_0603_1608Metric
- R_VDD1: renamed from R_VDD; value R -> 1k; footprint (none) -> Resistor_SMD:R_0603_1608Metric
- TH1: renamed from TH?; value Thermistor -> 103AT, 10k
- U1: renamed from U?; footprint (none) -> Package_SO:TSSOP-24_4.4x7.8mm_P0.65mm
Connections:
- net labels added: +5V
- wire segments 100 -> 111
- no-connect marks 0 -> 2

Commit message: assign thermistor footprint
Parts:
- R_CHG1: value R -> 1k
- R_DSG1: value R -> 4.5k
Changed lines of the file:
@@
 P 4450 3750
 F 0 "R_DSG1" H 4520 3796 50  0000 L CNN
-F 1 "R" H 4520 3705 50  0000 L CNN
+F 1 "4.5k" H 4520 3705 50  0000 L CNN
 F 2 "Resistor_SMD:R_0603_1608Metric" V 4380 3750 50  0001 C CNN
 F 3 "~" H 4450 3750 50  0001 C CNN
@@
 P 5300 3750
 F 0 "R_CHG1" H 5370 3796 50  0000 L CNN
-F 1 "R" H 5370 3705 50  0000 L CNN
+F 1 "1k" H 5370 3705 50  0000 L CNN
 F 2 "Resistor_SMD:R_0603_1608Metric" V 5230 3750 50  0001 C CNN
 F 3 "~" H 5300 3750 50  0001 C CNN

Commit message: still incorrect footprint for transistor
Parts:
- added Q_NMOS_CHG2, Q_NMOS_CHG3, Q_NMOS_CHG4: Q2, digikey-footprints:TO-252-3, symbol Device:Q_NMOS_DGS
- added Q_NMOS_DGS2, Q_NMOS_DGS3, Q_NMOS_DGS4: Q, digikey-footprints:TO-252-3, symbol Device:Q_NMOS_DGS
- Q_NMOS_CHG1, Q_NMOS_DGS1: footprint (none) -> digikey-footprints:TO-252-3
- TH1: footprint (none) -> Resistor_SMD:R_0201_0603Metric
Connections:
- wire segments 111 -> 120
Changed lines of the file:
@@
 F 0 "Q_NMOS_DGS1" V 4900 4400 50  0000 C CNN
 F 1 "Q" V 4991 4400 50  0000 C CNN
-F 2 "" H 4850 4500 50  0001 C CNN
+F 2 "digikey-footprints:TO-252-3" H 4850 4500 50  0001 C CNN
 F 3 "~" H 4650 4400 50  0001 C CNN
 	1    4650 4400
@@
 L Device:Q_NMOS_DGS Q_NMOS_CHG1
 U 1 1 5D2DE5B1
-P 5150 4400
-F 0 "Q_NMOS_CHG1" V 5400 4400 50  0000 C CNN
-F 1 "Q2" V 5491 4400 50  0000 C CNN
-F 2 "" H 5350 4500 50  0001 C CNN
-F 3 "~" H 5150 4400 50  0001 C CNN
-	1    5150 4400
+P 7900 4400
+F 0 "Q_NMOS_CHG1" V 8150 4400 50  0000 C CNN
+F 1 "Q2" V 8241 4400 50  0000 C CNN
+F 2 "digikey-footprints:TO-252-3" H 8100 4500 50  0001 C CNN
+F 3 "~" H 7900 4400 50  0001 C CNN
+	1    7900 4400
 	0    -1   1    0
 $EndComp
@@
 F 0 "TH1" V 6458 2750 50  0000 C CNN
 F 1 "103AT, 10k" V 6549 2750 50  0000 C CNN
-F 2 "" H 6700 2750 50  0001 C CNN
+F 2 "Resistor_SMD:R_0201_0603Metric" H 6700 2750 50  0001 C CNN
 F 3 "~" H 6700 2750 50  0001 C CNN
 	1    6700 2750
@@
 	6500 3350 6350 3350
 Wire Wire Line
-	6000 2950 6000 3350
-Wire Wire Line
 	6000 3350 6050 3350
 Wire Wire Line
@@
 Wire Wire Line
 	6400 3000 6550 3000
-Text GLabel 6650 4500 2    50   Input ~ 0
+Text GLabel 9200 4500 2    50   Input ~ 0
 PACK-
 $Comp
 L Device:R R_LD1
 U 1 1 5D33CBBE
-P 5900 3700
-F 0 "R_LD1" H 5970 3746 50  0000 L CNN
-F 1 "470k" H 5970 3655 50  0000 L CNN
-F 2 "Resistor_SMD:R_0603_1608Metric" V 5830 3700 50  0001 C CNN
-F 3 "~" H 5900 3700 50  0001 C CNN
-	1    5900 3700
-	1    0    0    -1
-$EndComp
-Wire Wire Line
-	5300 3150 5900 3150
-Wire Wire Line
-	5900 3150 5900 3550
-Wire Wire Line
-	5900 3850 5900 4500
-Wire Wire Line
-	5900 4500 6650 4500
+P 8450 3950
+F 0 "R_LD1" H 8520 3996 50  0000 L CNN
+F 1 "470k" H 8520 3905 50  0000 L CNN
+F 2 "Resistor_SMD:R_0603_1608Metric" V 8380 3950 50  0001 C CNN
+F 3 "~" H 8450 3950 50  0001 C CNN
+	1    8450 3950
+	1    0    0    -1
+$EndComp
 $Comp
 L Device:R R_DSG1
 U 1 1 5D343617
-P 4450 3750
-F 0 "R_DSG1" H 4520 3796 50  0000 L CNN
-F 1 "4.5k" H 4520 3705 50  0000 L CNN
-F 2 "Resistor_SMD:R_0603_1608Metric" V 4380 3750 50  0001 C CNN
-F 3 "~" H 4450 3750 50  0001 C CNN
-	1    4450 3750
+P 4450 3900
+F 0 "R_DSG1" H 4520 3946 50  0000 L CNN
+F 1 "4.5k" H 4520 3855 50  0000 L CNN
+F 2 "Resistor_SMD:R_0603_1608Metric" V 4380 3900 50  0001 C CNN
+F 3 "~" H 4450 3900 50  0001 C CNN
+	1    4450 3900
 	1    0    0    -1
 $EndComp
@@
 L Device:R R_CHG1
 U 1 1 5D34384D
-P 5300 3750
-F 0 "R_CHG1" H 5370 3796 50  0000 L CNN
-F 1 "1k" H 5370 3705 50  0000 L CNN
-F 2 "Resistor_SMD:R_0603_1608Metric" V 5230 3750 50  0001 C CNN
-F 3 "~" H 5300 3750 50  0001 C CNN
-	1    5300 3750
-	1    0    0    -1
-$EndComp
-Wire Wire Line
-	5300 3250 5300 3600
-Wire Wire Line
-	4450 3250 4450 3600
-Wire Wire Line
-	4450 3900 4450 4200
-Wire Wire Line
-	5300 3900 5300 4200
+P 6700 3950
+F 0 "R_CHG1" H 6770 3996 50  0000 L CNN
+F 1 "1k" H 6770 3905 50  0000 L CNN
+F 2 "Resistor_SMD:R_0603_1608Metric" V 6630 3950 50  0001 C CNN
+F 3 "~" H 6700 3950 50  0001 C CNN
+	1    6700 3950
+	1    0    0    -1
+$EndComp
 $Comp
 L Device:R R_GS2
 U 1 1 5D34B287
-P 5350 4350
-F 0 "R_GS2" H 5420 4396 50  0000 L CNN
-F 1 "1M" H 5420 4305 50  0000 L CNN
-F 2 "Resistor_SMD:R_0603_1608Metric" V 5280 4350 50  0001 C CNN
-F 3 "~" H 5350 4350 50  0001 C CNN
-	1    5350 4350
+P 8100 4350
+F 0 "R_GS2" H 8170 4396 50  0000 L CNN
+F 1 "1M" H 8170 4305 50  0000 L CNN
+F 2 "Resistor_SMD:R_0603_1608Metric" V 8030 4350 50  0001 C CNN
+F 3 "~" H 8100 4350 50  0001 C CNN
+	1    8100 4350
 	1    0    0    -1
 $EndComp
@@
 $EndComp
 Wire Wire Line
-	5300 4200 5350 4200
-Wire Wire Line
-	5300 4200 5150 4200
-Connection ~ 5300 4200
-Wire Wire Line
-	4650 4200 4450 4200
-Wire Wire Line
-	4450 4200 4400 4200
-Connection ~ 4450 4200
-Wire Wire Line
 	4450 4500 4400 4500
 $Comp
@@
 $EndComp
 Wire Wire Line
-	5350 4500 5900 4500
-Connection ~ 5350 4500
-Connection ~ 5900 4500
-Wire Wire Line
 	4400 4500 4300 4500
 Connection ~ 4400 4500
@@
 	3900 4500 1900 4500
 Connection ~ 3900 4500
-Wire Wire Line
-	4950 4500 4850 4500
 $Comp
 L Device:R R1
@@
 Wire Wire Line
 	3200 3650 3700 3650
+Wire Wire Line
+	6000 2950 6000 3350
+Connection ~ 8100 4500
+$Comp
+L Device:Q_NMOS_DGS Q_NMOS_CHG4
+U 1 1 5D44B8C3
+P 7500 4400
+F 0 "Q_NMOS_CHG4" V 7750 4400 50  0000 C CNN
+F 1 "Q2" V 7841 4400 50  0000 C CNN
+F 2 "digikey-footprints:TO-252-3" H 7700 4500 50  0001 C CNN
+F 3 "~" H 7500 4400 50  0001 C CNN
+	1    7500 4400
+	0    -1   1    0
+$EndComp
+$Comp
+L Device:Q_NMOS_DGS Q_NMOS_CHG3
+U 1 1 5D44B921
+P 7100 4400
+F 0 "Q_NMOS_CHG3" V 7350 4400 50  0000 C CNN
+F 1 "Q2" V 7441 4400 50  0000 C CNN
+F 2 "digikey-footprints:TO-252-3" H 7300 4500 50  0001 C CNN
+F 3 "~" H 7100 4400 50  0001 C CNN
+	1    7100 4400
+	0    -1   1    0
+$EndComp
+$Comp
+L Device:Q_NMOS_DGS Q_NMOS_CHG2
+U 1 1 5D44B97B
+P 6700 4400
+F 0 "Q_NMOS_CHG2" V 6950 4400 50  0000 C CNN
+F 1 "Q2" V 7041 4400 50  0000 C CNN
+F 2 "digikey-footprints:TO-252-3" H 6900 4500 50  0001 C CNN
+F 3 "~" H 6700 4400 50  0001 C CNN
+	1    6700 4400
+	0    -1   1    0
+$EndComp
+$Comp
+L Device:Q_NMOS_DGS Q_NMOS_DGS2
+U 1 1 5D44F779
+P 5050 4400
+F 0 "Q_NMOS_DGS2" V 5300 4400 50  0000 C CNN
+F 1 "Q" V 5391 4400 50  0000 C CNN
+F 2 "digikey-footprints:TO-252-3" H 5250 4500 50  0001 C CNN
+F 3 "~" H 5050 4400 50  0001 C CNN
+	1    5050 4400
+	0    1    1    0
+$EndComp
+$Comp
+L Device:Q_NMOS_DGS Q_NMOS_DGS3
+U 1 1 5D44F7D1
+P 5450 4400
+F 0 "Q_NMOS_DGS3" V 5700 4400 50  0000 C CNN
+F 1 "Q" V 5791 4400 50  0000 C CNN
+F 2 "digikey-footprints:TO-252-3" H 5650 4500 50  0001 C CNN
+F 3 "~" H 5450 4400 50  0001 C CNN
+	1    5450 4400
+	0    1    1    0
+$EndComp
+$Comp
+L Device:Q_NMOS_DGS Q_NMOS_DGS4
+U 1 1 5D44F833
+P 5850 4400
+F 0 "Q_NMOS_DGS4" V 6100 4400 50  0000 C CNN
+F 1 "Q" V 6191 4400 50  0000 C CNN
+F 2 "digikey-footprints:TO-252-3" H 6050 4500 50  0001 C CNN
+F 3 "~" H 5850 4400 50  0001 C CNN
+	1    5850 4400
+	0    1    1    0
+$EndComp
+Wire Wire Line
+	6050 4500 6500 4500
+Wire Wire Line
+	4650 4200 5050 4200
+Connection ~ 4650 4200
+Connection ~ 5050 4200
+Wire Wire Line
+	5050 4200 5450 4200
+Connection ~ 5450 4200
+Wire Wire Line
+	5450 4200 5850 4200
+Wire Wire Line
+	6700 4200 7100 4200
+Connection ~ 7900 4200
+Connection ~ 7100 4200
+Wire Wire Line
+	7100 4200 7500 4200
+Connection ~ 7500 4200
+Wire Wire Line
+	7500 4200 7900 4200
+Wire Wire Line
+	7900 4200 8100 4200
+Wire Wire Line
+	5300 3250 5300 3750
+Wire Wire Line
+	5300 3750 6700 3750
+Wire Wire Line
+	5300 3150 5800 3150
+Wire Wire Line
+	5800 3150 5800 3650
+Wire Wire Line
+	5800 3650 8450 3650
+Wire Wire Line
+	8100 4500 8450 4500
+Wire Wire Line
+	4400 4200 4450 4200
+Wire Wire Line
+	4450 3250 4450 3750
+Wire Wire Line
+	4450 4050 4450 4200
+Connection ~ 4450 4200
+Wire Wire Line
+	4450 4200 4650 4200
+Wire Wire Line
+	6700 4100 6700 4200
+Connection ~ 6700 4200
+Wire Wire Line
+	6700 3750 6700 3800
+Wire Wire Line
+	8450 3650 8450 3800
+Wire Wire Line
+	8450 4100 8450 4500
+Connection ~ 8450 4500
+Wire Wire Line
+	8450 4500 9200 4500
 $EndSCHEMATC
