File: SailbotBMS.sch (KiCad schematic (older format))
At the start: 35 parts, among them J1 Conn_01x05_Female, J2 Conn_01x02, J3 Conn_01x02, U1 BQ77915

Commit message: change footprint for transistors - maybe still not right
Parts:
- Q_NMOS_CHG1, Q_NMOS_CHG2, Q_NMOS_CHG3, Q_NMOS_CHG4, Q_NMOS_DGS1, Q_NMOS_DGS2, Q_NMOS_DGS3, Q_NMOS_DGS4: footprint digikey-footprints:TO-252-3 -> Package_TO_SOT_SMD:TO-252-3_TabPin2
- TH1: footprint Resistor_SMD:R_0201_0603Metric -> Resistor_SMD:R_0402_1005Metric
Changed lines of the file:
@@
 F 0 "Q_NMOS_DGS1" V 4900 4400 50  0000 C CNN
 F 1 "Q" V 4991 4400 50  0000 C CNN
-F 2 "digikey-footprints:TO-252-3" H 4850 4500 50  0001 C CNN
+F 2 "Package_TO_SOT_SMD:TO-252-3_TabPin2" H 4850 4500 50  0001 C CNN
 F 3 "~" H 4650 4400 50  0001 C CNN
 	1    4650 4400
@@
 F 0 "Q_NMOS_CHG1" V 8150 4400 50  0000 C CNN
 F 1 "Q2" V 8241 4400 50  0000 C CNN
-F 2 "digikey-footprints:TO-252-3" H 8100 4500 50  0001 C CNN
+F 2 "Package_TO_SOT_SMD:TO-252-3_TabPin2" H 8100 4500 50  0001 C CNN
 F 3 "~" H 7900 4400 50  0001 C CNN
 	1    7900 4400
@@
 F 0 "TH1" V 6458 2750 50  0000 C CNN
 F 1 "103AT, 10k" V 6549 2750 50  0000 C CNN
-F 2 "Resistor_SMD:R_0201_0603Metric" H 6700 2750 50  0001 C CNN
+F 2 "Resistor_SMD:R_0402_1005Metric" H 6700 2750 50  0001 C CNN
 F 3 "~" H 6700 2750 50  0001 C CNN
 	1    6700 2750
@@
 F 0 "Q_NMOS_CHG4" V 7750 4400 50  0000 C CNN
 F 1 "Q2" V 7841 4400 50  0000 C CNN
-F 2 "digikey-footprints:TO-252-3" H 7700 4500 50  0001 C CNN
+F 2 "Package_TO_SOT_SMD:TO-252-3_TabPin2" H 7700 4500 50  0001 C CNN
 F 3 "~" H 7500 4400 50  0001 C CNN
 	1    7500 4400
@@
 F 0 "Q_NMOS_CHG3" V 7350 4400 50  0000 C CNN
 F 1 "Q2" V 7441 4400 50  0000 C CNN
-F 2 "digikey-footprints:TO-252-3" H 7300 4500 50  0001 C CNN
+F 2 "Package_TO_SOT_SMD:TO-252-3_TabPin2" H 7300 4500 50  0001 C CNN
 F 3 "~" H 7100 4400 50  0001 C CNN
 	1    7100 4400
@@
 F 0 "Q_NMOS_CHG2" V 6950 4400 50  0000 C CNN
 F 1 "Q2" V 7041 4400 50  0000 C CNN
-F 2 "digikey-footprints:TO-252-3" H 6900 4500 50  0001 C CNN
+F 2 "Package_TO_SOT_SMD:TO-252-3_TabPin2" H 6900 4500 50  0001 C CNN
 F 3 "~" H 6700 4400 50  0001 C CNN
 	1    6700 4400
@@
 F 0 "Q_NMOS_DGS2" V 5300 4400 50  0000 C CNN
 F 1 "Q" V 5391 4400 50  0000 C CNN
-F 2 "digikey-footprints:TO-252-3" H 5250 4500 50  0001 C CNN
+F 2 "Package_TO_SOT_SMD:TO-252-3_TabPin2" H 5250 4500 50  0001 C CNN
 F 3 "~" H 5050 4400 50  0001 C CNN
 	1    5050 4400
@@
 F 0 "Q_NMOS_DGS3" V 5700 4400 50  0000 C CNN
 F 1 "Q" V 5791 4400 50  0000 C CNN
-F 2 "digikey-footprints:TO-252-3" H 5650 4500 50  0001 C CNN
+F 2 "Package_TO_SOT_SMD:TO-252-3_TabPin2" H 5650 4500 50  0001 C CNN
 F 3 "~" H 5450 4400 50  0001 C CNN
 	1    5450 4400
@@
 F 0 "Q_NMOS_DGS4" V 6100 4400 50  0000 C CNN
 F 1 "Q" V 6191 4400 50  0000 C CNN
-F 2 "digikey-footprints:TO-252-3" H 6050 4500 50  0001 C CNN
+F 2 "Package_TO_SOT_SMD:TO-252-3_TabPin2" H 6050 4500 50  0001 C CNN
 F 3 "~" H 5850 4400 50  0001 C CNN
 	1    5850 4400

Commit message: initial layout
Parts:
- renumbered R5 to R1, R4 to R2, R2 to R4, R1 to R5
Changed lines of the file:
@@
 Connection ~ 3900 4500
 $Comp
-L Device:R R1
+L Device:R R5
 U 1 1 5D386026
 P 2450 2050
-F 0 "R1" V 2243 2050 50  0000 C CNN
+F 0 "R5" V 2243 2050 50  0000 C CNN
 F 1 "33" V 2334 2050 50  0000 C CNN
 F 2 "Resistor_SMD:R_0603_1608Metric" V 2380 2050 50  0001 C CNN
@@
 $EndComp
 $Comp
-L Device:R R2
+L Device:R R4
 U 1 1 5D3860E4
 P 2450 2350
-F 0 "R2" V 2243 2350 50  0000 C CNN
+F 0 "R4" V 2243 2350 50  0000 C CNN
 F 1 "33" V 2334 2350 50  0000 C CNN
 F 2 "Resistor_SMD:R_0603_1608Metric" V 2380 2350 50  0001 C CNN
@@
 $EndComp
 $Comp
-L Device:R R4
+L Device:R R2
 U 1 1 5D38616A
 P 2450 2950
-F 0 "R4" V 2243 2950 50  0000 C CNN
+F 0 "R2" V 2243 2950 50  0000 C CNN
 F 1 "33" V 2334 2950 50  0000 C CNN
 F 2 "Resistor_SMD:R_0603_1608Metric" V 2380 2950 50  0001 C CNN
@@
 $EndComp
 $Comp
-L Device:R R5
+L Device:R R1
 U 1 1 5D3861AE
 P 2450 3250
-F 0 "R5" V 2243 3250 50  0000 C CNN
+F 0 "R1" V 2243 3250 50  0000 C CNN
 F 1 "33" V 2334 3250 50  0000 C CNN
 F 2 "Resistor_SMD:R_0603_1608Metric" V 2380 3250 50  0001 C CNN
