File: SailbotBMS.sch (KiCad schematic (older format))
At the start: 35 parts, among them J1 Conn_01x05_Female, J2 Conn_01x02, J3 Conn_01x02, U1 BQ77915

Commit message: afternoon check-in
Parts:
- R_OCD1: value R -> 196k
Changed lines of the file:
@@
 P 6250 3000
 F 0 "R_OCD1" V 6457 3000 50  0000 C CNN
-F 1 "R" V 6366 3000 50  0000 C CNN
+F 1 "196k" V 6366 3000 50  0000 C CNN
 F 2 "Resistor_SMD:R_0603_1608Metric" V 6180 3000 50  0001 C CNN
 F 3 "~" H 6250 3000 50  0001 C CNN
 	1    6250 3000
 	0    -1   -1   0
-$EndComp
-$Comp
-L power:GNDREF #PWR05
-U 1 1 5D32916E
-P 6550 3000
-F 0 "#PWR05" H 6550 2750 50  0001 C CNN
-F 1 "GNDREF" H 6555 2827 50  0000 C CNN
-F 2 "" H 6550 3000 50  0001 C CNN
-F 3 "" H 6550 3000 50  0001 C CNN
-	1    6550 3000
-	1    0    0    -1
 $EndComp
 $Comp
@@
 Wire Wire Line
 	8450 4500 9200 4500
+$Comp
+L power:GNDREF #PWR?
+U 1 1 5D413F68
+P 6550 3000
+F 0 "#PWR?" H 6550 2750 50  0001 C CNN
+F 1 "GNDREF" H 6555 2827 50  0000 C CNN
+F 2 "" H 6550 3000 50  0001 C CNN
+F 3 "" H 6550 3000 50  0001 C CNN
+	1    6550 3000
+	1    0    0    -1
+$EndComp
 $EndSCHEMATC

Commit message: real estate is valuable
Parts:
- renumbered Q_NMOS_CHG1 to CHG1, Q_NMOS_CHG4 to CHG2, Q_NMOS_CHG3 to CHG3, Q_NMOS_CHG2 to CHG4, Q_NMOS_DGS1 to DGS1, Q_NMOS_DGS2 to DGS2, Q_NMOS_DGS3 to DGS3, Q_NMOS_DGS4 to DGS4
Changed lines of the file:
@@
 $EndDescr
 $Comp
-L Device:Q_NMOS_DGS Q_NMOS_DGS1
+L Device:Q_NMOS_DGS DGS1
 U 1 1 5D24BC09
 P 4650 4400
-F 0 "Q_NMOS_DGS1" V 4900 4400 50  0000 C CNN
+F 0 "DGS1" V 4900 4400 50  0000 C CNN
 F 1 "Q" V 4991 4400 50  0000 C CNN
 F 2 "Package_TO_SOT_SMD:TO-252-3_TabPin2" H 4850 4500 50  0001 C CNN
@@
 $EndComp
 $Comp
-L Device:Q_NMOS_DGS Q_NMOS_CHG1
+L Device:Q_NMOS_DGS CHG1
 U 1 1 5D2DE5B1
 P 7900 4400
-F 0 "Q_NMOS_CHG1" V 8150 4400 50  0000 C CNN
+F 0 "CHG1" V 8150 4400 50  0000 C CNN
 F 1 "Q2" V 8241 4400 50  0000 C CNN
 F 2 "Package_TO_SOT_SMD:TO-252-3_TabPin2" H 8100 4500 50  0001 C CNN
@@
 Connection ~ 8100 4500
 $Comp
-L Device:Q_NMOS_DGS Q_NMOS_CHG4
+L Device:Q_NMOS_DGS CHG2
 U 1 1 5D44B8C3
 P 7500 4400
-F 0 "Q_NMOS_CHG4" V 7750 4400 50  0000 C CNN
+F 0 "CHG2" V 7750 4400 50  0000 C CNN
 F 1 "Q2" V 7841 4400 50  0000 C CNN
 F 2 "Package_TO_SOT_SMD:TO-252-3_TabPin2" H 7700 4500 50  0001 C CNN
@@
 $EndComp
 $Comp
-L Device:Q_NMOS_DGS Q_NMOS_CHG3
+L Device:Q_NMOS_DGS CHG3
 U 1 1 5D44B921
 P 7100 4400
-F 0 "Q_NMOS_CHG3" V 7350 4400 50  0000 C CNN
+F 0 "CHG3" V 7350 4400 50  0000 C CNN
 F 1 "Q2" V 7441 4400 50  0000 C CNN
 F 2 "Package_TO_SOT_SMD:TO-252-3_TabPin2" H 7300 4500 50  0001 C CNN
@@
 $EndComp
 $Comp
-L Device:Q_NMOS_DGS Q_NMOS_CHG2
+L Device:Q_NMOS_DGS CHG4
 U 1 1 5D44B97B
 P 6700 4400
-F 0 "Q_NMOS_CHG2" V 6950 4400 50  0000 C CNN
+F 0 "CHG4" V 6950 4400 50  0000 C CNN
 F 1 "Q2" V 7041 4400 50  0000 C CNN
 F 2 "Package_TO_SOT_SMD:TO-252-3_TabPin2" H 6900 4500 50  0001 C CNN
@@
 $EndComp
 $Comp
-L Device:Q_NMOS_DGS Q_NMOS_DGS2
+L Device:Q_NMOS_DGS DGS2
 U 1 1 5D44F779
 P 5050 4400
-F 0 "Q_NMOS_DGS2" V 5300 4400 50  0000 C CNN
+F 0 "DGS2" V 5300 4400 50  0000 C CNN
 F 1 "Q" V 5391 4400 50  0000 C CNN
 F 2 "Package_TO_SOT_SMD:TO-252-3_TabPin2" H 5250 4500 50  0001 C CNN
@@
 $EndComp
 $Comp
-L Device:Q_NMOS_DGS Q_NMOS_DGS3
+L Device:Q_NMOS_DGS DGS3
 U 1 1 5D44F7D1
 P 5450 4400
-F 0 "Q_NMOS_DGS3" V 5700 4400 50  0000 C CNN
+F 0 "DGS3" V 5700 4400 50  0000 C CNN
 F 1 "Q" V 5791 4400 50  0000 C CNN
 F 2 "Package_TO_SOT_SMD:TO-252-3_TabPin2" H 5650 4500 50  0001 C CNN
@@
 $EndComp
 $Comp
-L Device:Q_NMOS_DGS Q_NMOS_DGS4
+L Device:Q_NMOS_DGS DGS4
 U 1 1 5D44F833
 P 5850 4400
-F 0 "Q_NMOS_DGS4" V 6100 4400 50  0000 C CNN
+F 0 "DGS4" V 6100 4400 50  0000 C CNN
 F 1 "Q" V 6191 4400 50  0000 C CNN
 F 2 "Package_TO_SOT_SMD:TO-252-3_TabPin2" H 6050 4500 50  0001 C CNN
@@
 	6700 4200 7100 4200
 Connection ~ 7900 4200
-Connection ~ 7100 4200
-Wire Wire Line
-	7100 4200 7500 4200
-Connection ~ 7500 4200
-Wire Wire Line
-	7500 4200 7900 4200
 Wire Wire Line
 	7900 4200 8100 4200
@@
 Wire Wire Line
 	6700 4100 6700 4200
-Connection ~ 6700 4200
 Wire Wire Line
 	6700 3750 6700 3800
@@
 	1    0    0    -1
 $EndComp
+Connection ~ 6700 4200
+Wire Wire Line
+	7500 4200 7900 4200
+Connection ~ 7500 4200
+Wire Wire Line
+	7100 4200 7500 4200
+Connection ~ 7100 4200
 $EndSCHEMATC

Commit message: select the correct DPAK footprint and put the transistors in parallel, not series
Parts:
- added R_GSC2, R_GSC3, R_GSC4, R_GSD2, R_GSD3, R_GSD4: 1M, Resistor_SMD:R_0603_1608Metric, symbol Device:R
- CHG1: renamed from CHG4; footprint Package_TO_SOT_SMD:TO-252-3_TabPin2 -> Package_TO_SOT_SMD:TO-252-2
- CHG2: renamed from CHG3; footprint Package_TO_SOT_SMD:TO-252-3_TabPin2 -> Package_TO_SOT_SMD:TO-252-2
- CHG3: renamed from CHG2; footprint Package_TO_SOT_SMD:TO-252-3_TabPin2 -> Package_TO_SOT_SMD:TO-252-2
- CHG4: renamed from CHG1; footprint Package_TO_SOT_SMD:TO-252-3_TabPin2 -> Package_TO_SOT_SMD:TO-252-2
- DGS1, DGS2, DGS3, DGS4: footprint Package_TO_SOT_SMD:TO-252-3_TabPin2 -> Package_TO_SOT_SMD:TO-252-2
- R_SNS1: value 100m -> 5m
- renumbered R_GS2 to R_GSC1, R_GS1 to R_GSD1
Connections:
- wire segments 120 -> 161

Commit message: PACK- in our case is GNDREF
Connections:
- wire segments 161 -> 162
Changed lines of the file:
@@
 Connection ~ 8450 4500
 Wire Wire Line
-	8450 4500 9200 4500
+	8450 4500 9100 4500
 $Comp
 L power:GNDREF #PWR0102
@@
 Wire Wire Line
 	4650 5400 4650 6000
+$Comp
+L power:GNDREF #PWR?
+U 1 1 5D48496F
+P 9100 4500
+F 0 "#PWR?" H 9100 4250 50  0001 C CNN
+F 1 "GNDREF" H 9105 4327 50  0000 C CNN
+F 2 "" H 9100 4500 50  0001 C CNN
+F 3 "" H 9100 4500 50  0001 C CNN
+	1    9100 4500
+	1    0    0    -1
+$EndComp
+Connection ~ 9100 4500
+Wire Wire Line
+	9100 4500 9200 4500
 $EndSCHEMATC

Commit message: end of day commit
Parts:
- removed J3: Conn_01x02, Connector_PinHeader_2.54mm:PinHeader_1x02_P2.54mm_Vertical, symbol Connector_Generic:Conn_01x02
- CHG1, CHG2, CHG3, CHG4: value Q2 -> 4V
- DGS1, DGS2, DGS3, DGS4: value Q -> 4V
- R_CHG1: value 1k -> 0
- R_DSG1: value 4.5k -> 0
- R_SNS1: value 5m -> 4m
Connections:
- net labels removed: +5V, PRES
Changed lines of the file:
@@
 P 4850 4400
 F 0 "DGS1" V 5100 4400 50  0000 C CNN
-F 1 "Q" V 5191 4400 50  0000 C CNN
+F 1 "4V" V 5191 4400 50  0000 C CNN
 F 2 "Package_TO_SOT_SMD:TO-252-2" H 5050 4500 50  0001 C CNN
 F 3 "~" H 4850 4400 50  0001 C CNN
@@
 P 6700 6200
 F 0 "CHG4" V 6950 6200 50  0000 C CNN
-F 1 "Q2" V 7041 6200 50  0000 C CNN
+F 1 "4V" V 7041 6200 50  0000 C CNN
 F 2 "Package_TO_SOT_SMD:TO-252-2" H 6900 6300 50  0001 C CNN
 F 3 "~" H 6700 6200 50  0001 C CNN
@@
 Wire Wire Line
 	4000 2250 4450 2250
-Text GLabel 5300 2350 2    50   Input ~ 0
-PRES
 Wire Wire Line
 	5400 2250 5800 2250
@@
 $EndComp
 $Comp
-L Device:R R_DSG1
-U 1 1 5D343617
-P 4450 3900
-F 0 "R_DSG1" H 4520 3946 50  0000 L CNN
-F 1 "4.5k" H 4520 3855 50  0000 L CNN
-F 2 "Resistor_SMD:R_0603_1608Metric" V 4380 3900 50  0001 C CNN
-F 3 "~" H 4450 3900 50  0001 C CNN
-	1    4450 3900
-	1    0    0    -1
-$EndComp
-$Comp
-L Device:R R_CHG1
-U 1 1 5D34384D
-P 6700 3950
-F 0 "R_CHG1" H 6770 3996 50  0000 L CNN
-F 1 "1k" H 6770 3905 50  0000 L CNN
-F 2 "Resistor_SMD:R_0603_1608Metric" V 6630 3950 50  0001 C CNN
-F 3 "~" H 6700 3950 50  0001 C CNN
-	1    6700 3950
-	1    0    0    -1
-$EndComp
-$Comp
 L Device:R R_GSC1
 U 1 1 5D34B287
@@
 P 4150 4500
 F 0 "R_SNS1" V 3943 4500 50  0000 C CNN
-F 1 "5m" V 4034 4500 50  0000 C CNN
+F 1 "4m" V 4034 4500 50  0000 C CNN
 F 2 "Resistor_SMD:R_0603_1608Metric" V 4080 4500 50  0001 C CNN
 F 3 "~" H 4150 4500 50  0001 C CNN
@@
 Text GLabel 7600 3150 0    50   Input ~ 0
 PACK+
-$Comp
-L Connector_Generic:Conn_01x02 J3
-U 1 1 5D39668F
-P 7800 2050
-F 0 "J3" H 7880 2042 50  0000 L CNN
-F 1 "Conn_01x02" H 7880 1951 50  0000 L CNN
-F 2 "Connector_PinHeader_2.54mm:PinHeader_1x02_P2.54mm_Vertical" H 7800 2050 50  0001 C CNN
-F 3 "~" H 7800 2050 50  0001 C CNN
-	1    7800 2050
-	1    0    0    -1
-$EndComp
-Text GLabel 7600 2150 0    50   Input ~ 0
-PRES
-$Comp
-L power:+5V #PWR0101
-U 1 1 5D39678B
-P 7600 2050
-F 0 "#PWR0101" H 7600 1900 50  0001 C CNN
-F 1 "+5V" V 7615 2178 50  0000 L CNN
-F 2 "" H 7600 2050 50  0001 C CNN
-F 3 "" H 7600 2050 50  0001 C CNN
-	1    7600 2050
-	0    -1   -1   0
-$EndComp
 NoConn ~ 5300 2450
 NoConn ~ 5300 3050
@@
 P 6700 5600
 F 0 "CHG3" V 6950 5600 50  0000 C CNN
-F 1 "Q2" V 7041 5600 50  0000 C CNN
+F 1 "4V" V 7041 5600 50  0000 C CNN
 F 2 "Package_TO_SOT_SMD:TO-252-2" H 6900 5700 50  0001 C CNN
 F 3 "~" H 6700 5600 50  0001 C CNN
@@
 P 6700 5000
 F 0 "CHG2" V 6950 5000 50  0000 C CNN
-F 1 "Q2" V 7041 5000 50  0000 C CNN
+F 1 "4V" V 7041 5000 50  0000 C CNN
 F 2 "Package_TO_SOT_SMD:TO-252-2" H 6900 5100 50  0001 C CNN
 F 3 "~" H 6700 5000 50  0001 C CNN
@@
 P 6700 4400
 F 0 "CHG1" V 6950 4400 50  0000 C CNN
-F 1 "Q2" V 7041 4400 50  0000 C CNN
+F 1 "4V" V 7041 4400 50  0000 C CNN
 F 2 "Package_TO_SOT_SMD:TO-252-2" H 6900 4500 50  0001 C CNN
 F 3 "~" H 6700 4400 50  0001 C CNN
@@
 P 4850 5000
 F 0 "DGS2" V 5100 5000 50  0000 C CNN
-F 1 "Q" V 5191 5000 50  0000 C CNN
+F 1 "4V" V 5191 5000 50  0000 C CNN
 F 2 "Package_TO_SOT_SMD:TO-252-2" H 5050 5100 50  0001 C CNN
 F 3 "~" H 4850 5000 50  0001 C CNN
@@
 P 4850 5600
 F 0 "DGS3" V 5100 5600 50  0000 C CNN
-F 1 "Q" V 5191 5600 50  0000 C CNN
+F 1 "4V" V 5191 5600 50  0000 C CNN
 F 2 "Package_TO_SOT_SMD:TO-252-2" H 5050 5700 50  0001 C CNN
 F 3 "~" H 4850 5600 50  0001 C CNN
@@
 P 4850 6200
 F 0 "DGS4" V 5100 6200 50  0000 C CNN
-F 1 "Q" V 5191 6200 50  0000 C CNN
+F 1 "4V" V 5191 6200 50  0000 C CNN
 F 2 "Package_TO_SOT_SMD:TO-252-2" H 5050 6300 50  0001 C CNN
 F 3 "~" H 4850 6200 50  0001 C CNN
@@
 Wire Wire Line
 	5800 3650 8450 3650
-Wire Wire Line
-	4450 3250 4450 3750
-Wire Wire Line
-	4450 4050 4450 4200
-Wire Wire Line
-	6700 4100 6700 4200
-Wire Wire Line
-	6700 3750 6700 3800
 Wire Wire Line
 	8450 3650 8450 3800
@@
 	4650 5400 4650 6000
 $Comp
-L power:GNDREF #PWR?
+L power:GNDREF #PWR0103
 U 1 1 5D48496F
 P 9100 4500
-F 0 "#PWR?" H 9100 4250 50  0001 C CNN
+F 0 "#PWR0103" H 9100 4250 50  0001 C CNN
 F 1 "GNDREF" H 9105 4327 50  0000 C CNN
 F 2 "" H 9100 4500 50  0001 C CNN
@@
 Wire Wire Line
 	9100 4500 9200 4500
+Wire Wire Line
+	4450 4050 4450 4200
+Wire Wire Line
+	4450 3250 4450 3750
+Wire Wire Line
+	6700 3750 6700 3800
+Wire Wire Line
+	6700 4100 6700 4200
+$Comp
+L Device:R R_CHG1
+U 1 1 5D34384D
+P 6700 3950
+F 0 "R_CHG1" H 6770 3996 50  0000 L CNN
+F 1 "0" H 6770 3905 50  0000 L CNN
+F 2 "Resistor_SMD:R_0603_1608Metric" V 6630 3950 50  0001 C CNN
+F 3 "~" H 6700 3950 50  0001 C CNN
+	1    6700 3950
+	1    0    0    -1
+$EndComp
+$Comp
+L Device:R R_DSG1
+U 1 1 5D343617
+P 4450 3900
+F 0 "R_DSG1" H 4520 3946 50  0000 L CNN
+F 1 "0" H 4520 3855 50  0000 L CNN
+F 2 "Resistor_SMD:R_0603_1608Metric" V 4380 3900 50  0001 C CNN
+F 3 "~" H 4450 3900 50  0001 C CNN
+	1    4450 3900
+	1    0    0    -1
+$EndComp
+Text GLabel 5300 2350 2    50   Input ~ 0
+PACK+
 $EndSCHEMATC
